File: hardware/Pi Pico Module/GSED_0001/sensor_divider.kicad_sch (KiCad schematic)
At the start: 3 parts

Commit message: Reuploaded folder
Parts:
- C9: renamed from C1; footprint (none) -> CL10B104KB8NNNC:CAPC1608X90N; symbol Device:C -> CL10B104KB8NNNC:CL10B104KB8NNNC; A_max (none) -> 0.9; A_min (none) -> 0.9; A_nom (none) -> 0.9; D_max (none) -> 1.7; D_min (none) -> 1.5; D_nom (none) -> 1.6; E_max (none) -> 0.9; E_min (none) -> 0.7; E_nom (none) -> 0.8; L1_max (none) -> 0.5; L1_min (none) -> 0.1; L1_nom (none) -> 0.3; L_max (none) -> 0.5; L_min (none) -> 0.1; L_nom (none) -> 0.3; MANUFACTURER (none) -> Samsung Electro-Mechanics; STANDARD (none) -> IPC 7351B
- R6: footprint (none) -> TNPW060310K0BEEA:RESC1508X55N; symbol Device:R -> TNPW060310K0BEEA:TNPW060310K0BEEA
- R7: renamed from R1; footprint (none) -> TNPW060310K0BEEA:RESC1508X55N; symbol Device:R -> TNPW060310K0BEEA:TNPW060310K0BEEA
Connections:
- net GND: now also C9.1, R6.1; no longer C9.2, R6.2
- net Sigin: now also R7.2; no longer R7.1
- net Sigout: now also C9.2, R6.2, R7.1; no longer C9.1, R6.1, R7.2
