File: hardware/Pi Pico Module/GSED_0001/GSED_0001.kicad_pcb (KiCad board)
At the start: 2 copper layers, 173.5 x 126 mm, 40 parts, among them J10 Ignition E-Match, J11 QD E-Match, J12 Radio, J14 Power Input, J4 K-Bottle PT, J5 Load Cell + Amp, J6 Tank PT, J7 Current Sensor, J8 K-Bottle TC, J9 Fill Servo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

Commit message: Finished Board
Parts:
- added C1: 22 uF, Capacitor_SMD:C_0805_2012Metric, B.Cu at (203.9, 125.5)
- added C2: 22 uF, Capacitor_SMD:C_0805_2012Metric, B.Cu at (203.9, 119.0)
- added C9: 22 uF, Capacitor_SMD:C_0805_2012Metric, B.Cu at (203.9, 122.0)
- added G***: LOGO, RDT_Logo:RDT_Logo, F.Cu at (84.5, 42.0)
- moved C66 5.28 mm to (196.4, 122.5)
- moved J7 4.39 mm to (143.8, 118.0)
- moved C67 2.27 mm to (196.4, 127.0)
Routing:
- net +5V: track 256.1 -> 270.7 mm, vias 2 -> 3
- net GND: track 62.9 -> 55.4 mm, vias 4 -> 6
- net /GPIO15_INA237 SCL: track 13.8 -> 9.09 mm
- net /GPIO14_INA237 SDA: track 16.6 -> 11.9 mm
- net unconnected-(A1-AGND-Pad33): track 0.00 -> 3.59 mm
- net +13V: track 152.0 -> 153.1 mm
Other:
- board text added: "Current Sensor"
- board text added: "Fill Servo"
- board text added: "Ignition E-Match"
- board text added: "K-Bottle PT"
- board text added: "Load Cell + Amp"
- board text added: "Pi Pico Module Drew Wotawa 11/2025"
- board text added: "Power Input"
- board text added: "QD E-Match"
- board text added: "Radio"
- board text added: "Tank PT"
- board text added: "Thermocouple"
