File: hardware/Pi Pico Module/GSED_0001/buckconverter.kicad_sch (KiCad schematic)
At the start: 10 parts, among them U2 LMR33640ADDAR

Commit message: Reuploaded folder
Parts:
- removed CHF: 220 nF, symbol Device:C
- removed Cboot: 0.1uF, symbol Device:C
- removed Cin: 10 uF, symbol Device:C
- removed Cout2, Cout3, Cout4: 22 uF, symbol Device:C
- removed L1: 6.8 uH, symbol Device:L
- removed RFBT: 100K, symbol Device:R
- removed U2: LMR33640ADDAR, LMR33640ADDAR:VREG_LM5017MR_NOPB, symbol LMR33640ADDAR:LMR33640ADDAR
- added C12: DNP, Capacitor_SMD:C_0805_2012Metric, symbol Device:C
- added C6, C7, C8: 22 uF, Capacitor_SMD:C_0805_2012Metric, symbol Device:C
- added C66: 10u, Capacitor_SMD:C_0805_2012Metric, symbol Device:C
- added C67: 220n, Capacitor_SMD:C_0805_2012Metric, symbol Device:C
- added C69: 100n, Capacitor_SMD:C_0603_1608Metric, symbol Device:C
- added C72: 1u, Capacitor_SMD:C_0805_2012Metric, symbol Device:C
- added L2: 6.8 uH, CSBX0650_6R8M:IND_CSBX0650-6R8M, symbol Device:L
- added R3: 100K, Resistor_SMD:R_0603_1608Metric, symbol Device:R_US
- added R8: 24.9K, Resistor_SMD:R_0603_1608Metric, symbol Device:R_US
- added U3: LMR33640ADDAR, LMR33640ADDAR:VREG_LM5017MR_NOPB, symbol LMR33640ADDAR:LMR33640ADDAR
- C5: renamed from Cout1; footprint (none) -> Capacitor_SMD:C_0805_2012Metric; DigiKey (none) -> https://www.digikey.com/en/products/detail/samsung-electro-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
Connections:
- net GND: now also C6.2, C66.2, C67.2, C7.2, C72.2, C8.2, R8.2, U3.1 (AGND)
- net Vout renamed Vout (5V)
- net Vout (5V): now also C12.2, C6.1, C7.1, C8.1, L2.2, R3.2
- new net: C69.2, L2.1, U3.8 (SW)
- new net: C69.1, U3.7 (BOOT)
- new net: C72.1, U3.6 (VCC)
- new net: C12.1, R3.1, R8.1, U3.5 (FB)
- new net Vin (11.1V): C66.1, C67.1, U3.2 (VIN), U3.3 (EN)
- no-connect marks 2 -> 1
Other:
- note added: "F_sw = 400kHz I_outMax = 4A"
- note added: "Optional 0805 footprint. Implement if output unstable."
- note added: "Voltage Divider to regulate FB to 1V."
- moved on the sheet: C5

Commit message: Updated PCB
Connections:
- net Vout (5V) renamed +5V
Changed lines of the file:
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@@
+	)
+	(junction
+		(at 233.68 57.15)
+		(diameter 0)
+		(color 0 0 0 0)
 	)
 	(junction
@@
 	(wire
 		(pts
-			(xy 238.76 57.15) (xy 229.87 57.15)
+			(xy 238.76 57.15) (xy 233.68 57.15)
 		)
 		(stroke
@@
 		(pts
 			(xy 229.87 57.15) (xy 229.87 63.5)
+		)
+		(stroke
+			(width 0)
+			(type default)
+		)
+	)
+	(wire
+		(pts
+			(xy 233.68 57.15) (xy 229.87 57.15)
 		)
 		(stroke
@@
 					(unit 1)
 				)
+			)
+		)
+	)
+	(symbol
+		(lib_id "power:+5V")
+		(at 233.68 57.15 0)
+		(unit 1)
+		(exclude_from_sim no)
+		(in_bom yes)
+		(on_board yes)
+		(dnp no)
+		(fields_autoplaced yes)
+		(property "Reference" "#PWR037"
+			(at 233.68 60.96 0)
+			(effects
+				(font
+					(size 1.27 1.27)
+				)
+				(hide yes)
+			)
+		)
+		(property "Value" "+5V"
+			(at 233.68 52.07 0)
+			(effects
+				(font
+					(size 1.27 1.27)
+				)
+			)
+		)
+		(property "Footprint" ""
+			(at 233.68 57.15 0)
+			(effects
+				(font
+					(size 1.27 1.27)
+				)
+				(hide yes)
+			)
+		)
+		(property "Datasheet" ""
+			(at 233.68 57.15 0)
+			(effects
+				(font
+					(size 1.27 1.27)
+				)
+				(hide yes)
+			)
+		)
+		(property "Description" "Power symbol creates a global label with name \"+5V\""
+			(at 233.68 57.15 0)
+			(effects
+				(font
+					(size 1.27 1.27)
+				)
+				(hide yes)
+			)
+		)
+		(pin "1"
+		)
+		(instances
+			(project "GSED_0001"
+				(path "/264b8d8f-c165-4609-b867-e24f99960723/221c21bc-c9d9-4ebe-8506-48c1d255907f"
+					(reference "#PWR037")
+					(unit 1)
+				)

Commit message: Hopefully finished PCB
Parts:
- U3: footprint LMR33640ADDAR:VREG_LM5017MR_NOPB -> Package_SO:Texas_HSOP-8-1EP_3.9x4.9mm_P1.27mm_ThermalVias
Connections:
- net Vin (11.1V) renamed +13V
Changed lines of the file:
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@@
+	)
+	(junction
+		(at 43.18 60.96)
+		(diameter 0)
+		(color 0 0 0 0)
 	)
 	(junction
@@
 	(wire
 		(pts
-			(xy 41.91 60.96) (xy 45.72 60.96)
+			(xy 41.91 60.96) (xy 43.18 60.96)
 		)
 		(stroke
@@
 	(wire
 		(pts
+			(xy 43.18 60.96) (xy 45.72 60.96)
+		)
+		(stroke
+			(width 0)
+			(type default)
+		)
+	)
+	(wire
+		(pts
 			(xy 172.72 87.63) (xy 172.72 93.98)
 		)
@@
 		)
 	)
-	(hierarchical_label "Vin (11.1V)"
+	(hierarchical_label "Vin (13V)"
 		(shape input)
 		(at 41.91 60.96 180)
@@
 			)
 		)
-		(property "Footprint" "LMR33640ADDAR:VREG_LM5017MR_NOPB"
+		(property "Footprint" "Package_SO:Texas_HSOP-8-1EP_3.9x4.9mm_P1.27mm_ThermalVias"
 			(at 93.98 76.2 0)
 			(effects
@@
 					(unit 1)
 				)
+			)
+		)
+	)
+	(symbol
+		(lib_id "power:+12V")
+		(at 43.18 60.96 0)
+		(unit 1)
+		(exclude_from_sim no)
+		(in_bom yes)
+		(on_board yes)
+		(dnp no)
+		(fields_autoplaced yes)
+		(property "Reference" "#PWR03"
+			(at 43.18 64.77 0)
+			(effects
+				(font
+					(size 1.27 1.27)
+				)
+				(hide yes)
+			)
+		)
+		(property "Value" "+13V"
+			(at 43.18 55.88 0)
+			(effects
+				(font
+					(size 1.27 1.27)
+				)
+			)
+		)
+		(property "Footprint" ""
+			(at 43.18 60.96 0)
+			(effects
+				(font
+					(size 1.27 1.27)
+				)
+				(hide yes)
+			)
+		)
+		(property "Datasheet" ""
+			(at 43.18 60.96 0)
+			(effects
+				(font
+					(size 1.27 1.27)
+				)
+				(hide yes)
+			)
+		)
+		(property "Description" "Power symbol creates a global label with name \"+12V\""
+			(at 43.18 60.96 0)
+			(effects
+				(font
+					(size 1.27 1.27)
+				)
+				(hide yes)
+			)
+		)
+		(pin "1"
+		)
+		(instances
+			(project ""
+				(path "/264b8d8f-c165-4609-b867-e24f99960723/221c21bc-c9d9-4ebe-8506-48c1d255907f"
+					(reference "#PWR03")
+					(unit 1)
+				)

Commit message: Finished Board
Parts:
- added C1, C2, C9: 22 uF, Capacitor_SMD:C_0805_2012Metric, symbol Device:C
Connections:
- net +5V: now also C1.1, C2.1, C9.1
- net GND: now also C1.2, C2.2, C9.2
Other:
- moved on the sheet: C12, C5, C6, C66, C67, C69, C7, C72, C8, L2, R3, R8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
