File: hardware/Pi Pico Module/GSED_0001/buckconverter.kicad_sch (KiCad schematic)
At the start: 13 parts, among them U3 LMR33640ADDAR

Commit message: Done
Parts:
- removed C66: 10u, Capacitor_SMD:C_0805_2012Metric, symbol Device:C
- removed C67: 220n, Capacitor_SMD:C_0805_2012Metric, symbol Device:C
- removed C69: 100n, Capacitor_SMD:C_0603_1608Metric, symbol Device:C
- removed C72: 1u, Capacitor_SMD:C_0805_2012Metric, symbol Device:C
- added C15, C16, C17: 22 uF, Capacitor_SMD:C_0805_2012Metric, symbol Device:C
- added C18, C19: 10u, Capacitor_SMD:C_1210_3225Metric, symbol Device:C
- added C20: 220n, Capacitor_SMD:C_0805_2012Metric, symbol Device:C
- added C21: 1u, Capacitor_SMD:C_0805_2012Metric, symbol Device:C
- added C22: 100n, Capacitor_SMD:C_0603_1608Metric, symbol Device:C
- added R10: 2.49k, Resistor_SMD:R_0603_1608Metric, symbol Device:R_US
- added R11: 10K, Resistor_SMD:R_0603_1608Metric, symbol Device:R_US
- U3: footprint Package_SO:Texas_HSOP-8-1EP_3.9x4.9mm_P1.27mm_ThermalVias -> LMR33640ADDAR:VREG_LM5017MR_NOPB
Connections:
- net +13V: now also C18.1, C19.1, C20.1, R11.1; no longer U3.3 (EN)
- net +5V: now also C15.1, C16.1, C17.1
- net GND: now also U3.9 (AGND), C15.2, C16.2, C17.2, C18.2, C19.2, C20.2, C21.2, R10.1
- net SW: now reaches L2.1, U3.8 (SW)
- net SW: now also C22.2
- net at U3.7 (BOOT): now also C22.1
- net at U3.6 (VCC): now also C21.1
- net FB: now reaches C12.1, R3.1, R8.1, U3.5 (FB)
- new net: R10.2, R11.2, U3.3 (EN)
Other:
- moved on the sheet: C6, C7, C8, U3
