File: hardware/Pi Pico Module/GSED_0001/GSED_0001.kicad_sch (KiCad schematic)
At the start: 17 parts, among them J1 Conn_01x10_Socket, J10 Ignition E-Match, J11 QD E-Match, J12 Radio, J14 Power Input, J2 Conn_01x10_Socket, J3 Conn_01x10_Socket (Digital), J4 K-Bottle PT, J5 Load Cell + Amp, J6 Tank PT, J7 Current Sensor, J8 K-Bottle TC, J9 Fill Servo, U1 BA90BC0FP-E2

Commit message: Reuploaded folder
Parts:
- added C10, C11, C13: 100n, Capacitor_SMD:C_0603_1608Metric, symbol Device:C
- added C14: 150u, EEUFC1H151B:CAPPRD500W60D1000H1600, symbol Device:C_Polarized
- added D1: 1N5817, Diode_THT:D_DO-41_SOD81_P10.16mm_Horizontal, symbol Diode:1N5817
- added R10, R9: 1k, Resistor_SMD:R_0603_1608Metric, symbol Device:R_US
- C3: footprint (none) -> Capacitor_SMD:C_0805_2012Metric; symbol Device:C -> 595D226X0050R2T:595D226X0050R2T
- C4: footprint (none) -> TAJA334K050RNJ:CAPMP3216X180N; symbol Device:C -> TAJA334K050RNJ:TAJA334K050RNJ; MANUFACTURER (none) -> AVX; MAXIMUM_PACKAGE_HEIGHT (none) -> 1.8 mm; PARTREV (none) -> 031320; STANDARD (none) -> IPC 7351B
- J1, J2, J3: footprint (none) -> Connector_PinHeader_2.54mm:PinHeader_1x10_P2.54mm_Vertical
- J10, J11, J4, J6, J9: footprint (none) -> Connector_PinHeader_2.54mm:PinHeader_1x03_P2.54mm_Vertical
- J12, J5, J7: footprint (none) -> Connector_PinHeader_2.54mm:PinHeader_1x04_P2.54mm_Vertical
- J14: footprint (none) -> Connector_AMASS:AMASS_XT30U-M_1x02_P5.0mm_Vertical
- J8: footprint (none) -> AM-K-PCB:AMKPCB
Connections:
- net Vin (DAQ_Module5V) is gone; now on net +5V: J1.7 (Pin_7)
- net +13V: now also C4.1, C10.2, C11.2, C13.2, C14.1; no longer C4.2, J12.1 (Pin_1)
- net +5V: now also A1.37 (3V3_EN), J12.1 (Pin_1)
- net +9V: now also C3.1; no longer C3.2
- net GND: now also C3.2, C4.2, C10.1, C11.1, C13.1, C14.2; no longer C3.1, C4.1
- net GPIO0 (Ignition_E-Match): now also R9.1; no longer A1.1 (GPIO0)
- net GPIO1 (QD_E-Match): now also R10.1; no longer A1.2 (GPIO1)
- net at A1.39 (VSYS): now also D1.1 (K)
- new net: A1.1 (GPIO0), R9.2
- new net: A1.2 (GPIO1), R10.2
- no-connect marks 2 -> 1
Other:
- company: (none) -> Rocket Design Team
- title: (none) -> Pi Pico Module
- moved on the sheet: A1, J1, J10, J11, J12, J14, J2, J3, J4, J5, J6, J7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

Commit message: Updated PCB
Parts:
- removed J1, J2: Conn_01x10_Socket, Connector_PinHeader_2.54mm:PinHeader_1x10_P2.54mm_Vertical, symbol Connector:Conn_01x10_Socket
- removed R10, R9: 1k, Resistor_SMD:R_0603_1608Metric, symbol Device:R_US
- added J13: Conn_01x20_Socket, Connector_PinHeader_2.54mm:PinHeader_1x20_P2.54mm_Vertical, symbol Connector:Conn_01x20_Socket
- added R1, R2: 1k, Resistor_SMD:R_0603_1608Metric, symbol Device:R_US
Connections:
- net Divider+LowPass1/Sigin is gone; now on net ADC_AI0: J4.2 (Pin_2)
- net Divider+LowPass2/Sigin is gone; now on net ADC_AI1: J6.2 (Pin_2)
- net Divider+LowPass3/Sigin is gone; now on net ADC_AI2: J5.2 (Pin_2)
- net +5V: now also J13.20 (Pin_20)
- net ADC_AI0: now also J13.1 (Pin_1)
- net ADC_AI1: now also J13.2 (Pin_2)
- net ADC_AI2: now also J13.3 (Pin_3)
- net ADC_AI3: now also J13.4 (Pin_4)
- net ADC_AI4: now also J13.5 (Pin_5)
- net ADC_AI5: now also J13.6 (Pin_6)
- net ADC_AI6: now also J13.7 (Pin_7)
- net ADC_AI7: now also J13.8 (Pin_8)
- net GND: now also J13.16 (Pin_16), J13.17 (Pin_17), J13.18 (Pin_18), J13.19 (Pin_19), J13.9 (Pin_9)
- net T+ (ChamberShell_1): now also J13.10 (Pin_10)
- net T+ (ChamberShell_2): now also J13.12 (Pin_12)
- net T+ (N2O): now also J13.14 (Pin_14)
- net T- (ChamberShell_1): now also J13.11 (Pin_11)
- net T- (ChamberShell_2): now also J13.13 (Pin_13)
- net T- (N2O): now also J13.15 (Pin_15)
- net GPIO18 (Fill Servo): now reaches A1.24 (GPIO18)
- net GPIO18 (Fill Servo): now also J9.2 (Pin_2)
- net at A1.25 (GPIO19): now also R2.2
- net at A1.26 (GPIO20): now also R1.2
- net GPIO0 (Ignition_E-Match) renamed GPIO20 (Ignition_E-Match)
- net GPIO20 (Ignition_E-Match): now also R1.1
- net GPIO1 (QD_E-Match) renamed GPIO19 (QD_E-Match)
- net GPIO19 (QD_E-Match): now also R2.1
- net GPIO2 (Fill Servo): no longer names the net of A1.4 (GPIO2)
- net GPIO2 (Fill Servo): no longer J9.2 (Pin_2)
Other:
- removed sheet Divider+LowPass1
- removed sheet Divider+LowPass2
- removed sheet Divider+LowPass3

Commit message: Hopefully finished PCB
Parts:
- removed J13: Conn_01x20_Socket, Connector_PinHeader_2.54mm:PinHeader_1x20_P2.54mm_Vertical, symbol Connector:Conn_01x20_Socket
- removed J3: Conn_01x10_Socket (Digital), Connector_PinHeader_2.54mm:PinHeader_1x10_P2.54mm_Vertical, symbol Connector:Conn_01x10_Socket
- added D2: 1N5817, Diode_THT:D_DO-41_SOD81_P10.16mm_Horizontal, symbol Diode:1N5817
- added U2: ~, DAQ_Module:DAQ_Module, symbol DAQ_Module:DAQ_Module
Connections:
- net +5V: now also D1.2 (A), D2.1 (K), U2.11 (Vin_(5V)); no longer A1.37 (3V3_EN)
- net ADC_AI0: now also U2.8 (ADC_AI7)
- net ADC_AI1: now also U2.7 (ADC_AI6)
- net ADC_AI2: now also U2.6 (ADC_AI5)
- net ADC_AI3: now also U2.5 (ADC_AI4)
- net ADC_AI4: now also U2.4 (ADC_AI3)
- net ADC_AI5: now also U2.3 (ADC_AI2)
- net ADC_AI6: now also U2.2 (ADC_AI1)
- net ADC_AI7: now also U2.1 (ADC_AI0)
- net GND: now also U2.10 (GND), U2.12 (GND), U2.13 (GND), U2.20 (GND), U2.30 (GND), U2.9 (GND)
- net GPIO10 (SCK_TCIC): now also U2.27 (SCK_TCIC)
- net GPIO12 (CS_N2O): now also U2.29 (CS_TCIC3)
- net GPIO13 (CSChamberShell_2): now also U2.28 (CS_TCIC2)
- net GPIO4 (MISO_ADC): now also U2.21 (MISO_ADC)
- net GPIO5 (CS_ADC): now also U2.24 (CS_ADC)
- net GPIO6 (SCK_ADC): now also U2.23 (SCK_ADC)
- net GPIO7 (MOSI_ADC): now also U2.22 (MOSI_ADC)
- net GPIO8 (MISO_TCIC): now also U2.25 (MISO_TCIC)
- net GPIO9 (CSChamberShell_1): now also U2.26 (CS_TCIC1)
- net T+ (ChamberShell_1): now also U2.15 (T1+)
- net T+ (ChamberShell_2): now also U2.17 (T2+)
- net T+ (N2O): now also U2.19 (T3+)
- net T- (ChamberShell_1): now also U2.14 (T1-)
- net T- (ChamberShell_2): now also U2.16 (T2-)
- net T- (N2O): now also U2.18 (T3-)
- new net: A1.37 (3V3_EN), D2.2 (A)

Commit message: Done
Parts:
- removed C3: 22 uF, Capacitor_SMD:C_0805_2012Metric, symbol 595D226X0050R2T:595D226X0050R2T
- removed C4: 0.33 uF, TAJA334K050RNJ:CAPMP3216X180N, symbol TAJA334K050RNJ:TAJA334K050RNJ
- removed J4: K-Bottle PT, Connector_PinHeader_2.54mm:PinHeader_1x03_P2.54mm_Vertical, symbol Connector_Generic:Conn_01x03
- removed J5: Load Cell + Amp, Connector_PinHeader_2.54mm:PinHeader_1x04_P2.54mm_Vertical, symbol Connector_Generic:Conn_01x04
- removed U1: BA90BC0FP-E2, TO252-3_ROM, symbol BA90BC0FP-E2:BA90BC0FP-E2
- added C1, C2, C3, C9: 100n, Capacitor_SMD:C_0603_1608Metric, symbol Device:C
- added C23: 0.33u, Capacitor_SMD:C_1206_3216Metric, symbol Device:C
- added J1: N2-Bottle PT, TerminalBlock:TerminalBlock_Xinya_XY308-2.54-3P_1x03_P2.54mm_Horizontal, symbol Connector_Generic:Conn_01x03
- added J13: Purge Servo, TerminalBlock:TerminalBlock_Xinya_XY308-2.54-3P_1x03_P2.54mm_Horizontal, symbol Connector_Generic:Conn_01x03
- added J15: Internal Cooling, Connector_PinHeader_2.54mm:PinHeader_1x03_P2.54mm_Vertical, symbol Connector_Generic:Conn_01x03
- added J16: Nitrous Cooling, Connector_PinHeader_2.54mm:PinHeader_1x03_P2.54mm_Vertical, symbol Connector_Generic:Conn_01x03
- added J17: Load Cell + Amp, TerminalBlock:TerminalBlock_Xinya_XY308-2.54-3P_1x03_P2.54mm_Horizontal, symbol Connector_Generic:Conn_01x03
- added J2, J3: K-Bottle TC, TerminalBlock:TerminalBlock_Xinya_XY308-2.54-2P_1x02_P2.54mm_Horizontal, symbol Connector_Generic:Conn_01x02
- added J5: K-Bottle PT, TerminalBlock:TerminalBlock_Xinya_XY308-2.54-3P_1x03_P2.54mm_Horizontal, symbol Connector_Generic:Conn_01x03
- added Q1: BUK6Y33-60PX, BUK6Y33-60PX:LFPAK_SOT669_NEX, symbol BUK6Y33-60PX:BUK6Y33-60PX
- added Q3: Q_NPN, Package_TO_SOT_SMD:SOT-323_SC-70, symbol Device:Q_NPN
- added R12, R13, R5, R6: 2.49k, Resistor_SMD:R_0603_1608Metric, symbol Device:R_US
- added R4: 1k, Resistor_SMD:R_1206_3216Metric, symbol Device:R_US
- added R7, R9: 10K, Resistor_SMD:R_0603_1608Metric, symbol Device:R_US
- added U1: L78M09CDT-TR, Package_TO_SOT_SMD:TO-252-2, symbol L78M09CDT-TR:L78M09CDT-TR
- added U4, U5: BAV199_215, BAV199_215:TO-236AB_NEX, symbol BAV199_215:BAV199_215
- J12: value Radio -> Radio Module Connector
- J6, J9: footprint Connector_PinHeader_2.54mm:PinHeader_1x03_P2.54mm_Vertical -> TerminalBlock:TerminalBlock_Xinya_XY308-2.54-3P_1x03_P2.54mm_Horizontal
- J8: footprint AM-K-PCB:AMKPCB -> TerminalBlock:TerminalBlock_Xinya_XY308-2.54-2P_1x02_P2.54mm_Horizontal
- U2: value ~ -> DAQ_Module
Connections:
- net ADC_AI4 is gone; now on net ADC_AI3: U2.4 (ADC_AI3)
- net ADC_AI5 is gone; now on net ADC_AI2: U2.3 (ADC_AI2)
- net ADC_AI6 is gone; now on net ADC_AI1: U2.2 (ADC_AI1)
- net ADC_AI7 is gone; now on net ADC_AI0: U2.1 (ADC_AI0)
- net +13V: now also C11.1, C13.1, J10.2 (Pin_2), J11.2 (Pin_2), J14.2 (Pin_2), C2.1, C23.2, C9.1, J15.2 (Pin_2), J16.2 (Pin_2), J17.1 (Pin_1), Q1.1 (S), Q1.2 (S), Q1.3 (S), R9.1, U1.1 (IN); no longer C10.2, C11.2, C13.2, J10.1 (Pin_1), J11.1 (Pin_1), J14.1 (Pin_1), J9.1 (Pin_1)
- net +9V: now also C3.2, J1.1 (Pin_1), J5.1 (Pin_1), R4.1, U1.3 (OUT)
- net ADC_AI0: now also J5.2 (Pin_2); no longer U2.8 (ADC_AI7)
- net ADC_AI1: no longer U2.7 (ADC_AI6)
- net ADC_AI2: now also J1.2 (Pin_2); no longer U2.6 (ADC_AI5)
- net ADC_AI3: now also J17.2 (Pin_2); no longer U2.5 (ADC_AI4)
- net GND: now also A1.33 (AGND), C10.2, C11.2, C13.2, J10.1 (Pin_1), J11.1 (Pin_1), J14.1 (Pin_1), J9.1 (Pin_1), C1.1, C2.2, C23.1, C3.1, C9.2, J1.3 (Pin_3), J13.3 (Pin_3), J15.1 (Pin_1), J16.1 (Pin_1), J17.3 (Pin_3), J5.3 (Pin_3), Q3.2 (E), R4.2, U1.2 (GND), U4.1, U5.1; no longer C10.1, C11.1, C13.1, J10.3 (Pin_3), J11.3 (Pin_3), J14.2 (Pin_2), J9.3 (Pin_3)
- net T+ (N2O): now also J8.2 (Pin_2); no longer J8.1 (Pin_1)
- net T- (N2O): now also J8.1 (Pin_1); no longer J8.2 (Pin_2)
- net GPIO0 (Radio_UART_TX): now reaches A1.1 (GPIO0)
- net GPIO0 (Radio_UART_TX): now also J12.2 (Pin_2)
- net GPIO1 (Radio_UART_RX): now reaches A1.2 (GPIO1)
- net GPIO1 (Radio_UART_RX): now also J12.3 (Pin_3)
- net at A1.25 (GPIO19): no longer R2.2
- net at R1.2: now also A1.32 (GPIO27_ADC1), U4.3; no longer A1.26 (GPIO20)
- net GPIO22 (Ignition_E-Match): now reaches A1.29 (GPIO22)
- net GPIO22 (Ignition_E-Match): now also R13.1
- net at A1.31 (GPIO26_ADC0): now also R2.2, U5.3
- net GPIO28 (ServoPWR_Switch): now reaches A1.34 (GPIO28_ADC2)
- net GPIO28 (ServoPWR_Switch): now also R7.2
- net +3.3V: now reaches A1.36 (3V3)
- net +3.3V: now also U4.2, U5.2
- net GPIO2_INA237 SDA: now reaches A1.4 (GPIO2)
- net GPIO2_INA237 SDA: now also J7.2 (Pin_2)
- net GPIO3_INA237 SCL: now reaches A1.5 (GPIO3)
- net GPIO3_INA237 SCL: now also J7.3 (Pin_3)
- net GPIO13 (CSChamberShell_2) renamed GPIO13 (CS_Internal)
- net GPIO14_INA237 SDA: no longer names the net of A1.19 (GPIO14)
- net GPIO14_INA237 SDA: no longer J7.2 (Pin_2)
- net GPIO15_INA237 SCL: no longer names the net of A1.20 (GPIO15)
- net GPIO15_INA237 SCL: no longer J7.3 (Pin_3)
- net GPIO16 (UART_TX) renamed GPIO16 (Nitrous_Cooling)
- net GPIO16 (Nitrous_Cooling): now also R5.1; no longer J12.2 (Pin_2)
- net GPIO17 (UART_RX): no longer names the net of A1.22 (GPIO17)
- net GPIO17 (UART_RX): no longer J12.3 (Pin_3)
- net GPIO18 (Fill Servo) renamed GPIO18 (Internal_Cooling)
- net GPIO18 (Internal_Cooling): now also R6.1; no longer J9.2 (Pin_2)
- net GPIO19 (QD_E-Match) renamed GPIO26 (Fill Servo)
- net GPIO26 (Fill Servo): now also J9.2 (Pin_2); no longer J11.2 (Pin_2)
- net GPIO20 (Ignition_E-Match) renamed GPIO27 (Purge Servo)
- net GPIO27 (Purge Servo): now also J13.2 (Pin_2); no longer J10.2 (Pin_2)
- net GPIO9 (CSChamberShell_1) renamed GPIO9 (CS_N2)
- net T+ (ChamberShell_1) renamed T+ (N2)
- net T+ (N2): now also J3.2 (Pin_2)
- net T+ (ChamberShell_2) renamed T+ (Internal)
- net T+ (Internal): now also J2.2 (Pin_2)
- net T- (ChamberShell_1) renamed T- (N2)
- net T- (N2): now also J3.1 (Pin_1)
- net T- (ChamberShell_2) renamed T- (Internal)
- net T- (Internal): now also J2.1 (Pin_1)
- new net: Q1.4 (G), Q3.3 (C), R9.2
- new net: J11.3 (Pin_3), R12.2
- new net: J16.3 (Pin_3), R5.2
- new net: J15.3 (Pin_3), R6.2
- new net: Q3.1 (B), R7.1
- new net: J10.3 (Pin_3), R13.2
- new net +V_Servo: C1.2, C10.1, J13.1 (Pin_1), J9.3 (Pin_3), Q1.5 (D)
- new net GPIO20 (QD_E-Match): A1.26 (GPIO20), R12.1
- no-connect marks 1 -> 12
Other:
- note added: "1206 Resistor footprint, for if LDO is unstable under low load. 200 Ohm selected for a 50mA load, experiment with different values if needed."
- note added: "DAQ Module"
- note added: "Outputs and Effector Control"
- note added: "Pi Pico (Microcontroller)"
- note added: "Power Input and Regulation"
- note added: "Radio Module Connection"
- note added: "Sensor Input"
- moved on the sheet: A1, C10, C11, C13, C14, D1, D2, J10, J11, J12, J14, J6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
