File: hardware/PDN Schematic/PDN Schematic.kicad_pcb (KiCad board)
At the start: 2 copper layers, 59.4 x 69.6 mm, 16 parts, among them J1 Conn_01x02_Pin, J10 Conn_01x02_Pin, J11 Led Indicator Pin, J2 Conn_01x02_Pin, J3 Conn_01x02_Pin, J4 Conn_01x04_Pin, J7 Conn_01x02_Pin, J8 Conn_01x02_Pin, J9 Conn_01x02_Pin, U1 Current Reader

Commit message: Extra GSE PDN Board changes
Parts:
- added G***: LOGO, RDT_Logo:RDT_Logo, F.Cu at (175.0, 106.0)
- moved J10 14.0 mm to (202.5, 38.0)
- moved REF** 13.2 mm to (209.0, 32.0)
- moved REF** 12.2 mm to (157.0, 32.0)
- moved R1 11.3 mm to (163.0, 87.0), turned to 90 degrees
- moved J9 10.5 mm to (202.3, 50.0)
- moved J4 7.58 mm to (186.5, 37.0)
- moved C1 7.58 mm to (178.7, 69.2)
- moved J1 7.58 mm to (163.3, 79.4)
- moved J11 7.58 mm to (163.2, 95.8)
- moved U1 7.58 mm to (186.9, 45.4)
- moved J8 6.97 mm to (202.0, 62.0)
- moved REF** 3.31 mm to (209.0, 104.0)
- moved J7 3.15 mm to (202.0, 74.4)
- moved J2 2.28 mm to (202.0, 98.0)
- moved REF** 1.73 mm to (157.0, 104.0)
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Connections:
- net Net-(J4-Pin_2) renamed GND2
Routing:
- net +13V: track 24.9 -> 0.00 mm
- net VOUT: track 11.5 -> 0.55 mm
- net Net-(J11-Pin_1): track 8.47 -> 7.39 mm
Other:
- board size 59.4 x 69.6 mm -> 66 x 86 mm
- board text added: "GSE PDN Board Britney Choimah 10/19/2025"

Commit message: proper library pathing
Parts:
- U1: footprint RocketDesignCustomFootprints:INA238_MODULE -> GSE_PDN_LIB:INA238_MODULE
- moved J4 0.52 mm to (187.0, 37.0)
Changed lines of the file:
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@@
 	(footprint "Connector_PinHeader_2.54mm:PinHeader_1x04_P2.54mm_Vertical"
 		(layer "F.Cu")
-		(at 186.4754 36.98 -90)
+		(at 187 36.98 -90)
 		(descr "Through hole straight pin header, 1x04, 2.54mm pitch, single row")
 		(tags "Through hole pin header THT 1x04 2.54mm single row")
@@
 		(embedded_fonts no)
 	)
-	(footprint "RocketDesignCustomFootprints:INA238_MODULE"
+	(footprint "GSE_PDN_LIB:INA238_MODULE"
 		(layer "F.Cu")
 		(at 186.89 45.405957 -90)
@@
 		)
 		(property "Value" "Current Reader"
-			(at 0 20.16 90)
-			(layer "F.Fab")
+			(at 0 20.16 270)
+			(layer "F.Fab")
+			(hide yes)
 			(effects
 				(font
@@
 		)
 		(property "Datasheet" ""
-			(at 0 0 90)
+			(at 0 0 270)
 			(layer "F.Fab")
 			(hide yes)
@@
 		)
 		(property "Description" ""
-			(at 0 0 90)
+			(at 0 0 270)
 			(layer "F.Fab")
 			(hide yes)
@@
 			)
 			(layer "F.SilkS")
-		)
-		(fp_text user "${REFERENCE}"
-			(at 0 8.89 0)
-			(layer "F.Fab")
-			(effects
-				(font
-					(size 1 1)
-					(thickness 0.15)
-				)
-			)
 		)
 		(pad "1" thru_hole circle
@@
 	)
 	(gr_text "GSE PDN Board\nBritney Choimah\n10/19/2025"
-		(at 192 110 0)
+		(at 191 108 0)
 		(layer "F.SilkS")
 		(effects
@@
 	)
 	(segment
-		(start 186.9154 37.42)
-		(end 186.4754 36.98)
+		(start 186.9154 45.38)
+		(end 186.9154 37.42)
 		(width 0.4)
 		(layer "F.Cu")
@@
 	)
 	(segment
-		(start 186.9154 45.38)
-		(end 186.9154 37.42)
+		(start 186.9154 37.42)
+		(end 186.4754 36.98)
 		(width 0.4)
 		(layer "F.Cu")
