File: hardware/GSECPM/buckconverter.kicad_sch (KiCad schematic)
At the start: 19 parts, among them U3 LMR33640ADDAR

Commit message: Made all buck components on front layer
Parts:
- U3: footprint LMR33640ADDAR:VREG_LM5017MR_NOPB -> Package_SO:Texas_HSOP-8-1EP_3.9x4.9mm_P1.27mm_ThermalVias
Changed lines of the file:
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@@
 			)
 		)
-		(property "Footprint" "LMR33640ADDAR:VREG_LM5017MR_NOPB"
+		(property "Footprint" "Package_SO:Texas_HSOP-8-1EP_3.9x4.9mm_P1.27mm_ThermalVias"
 			(at 97.79 76.2 0)
 			(effects
