File: hardware/GSECPM/buckconverter.kicad_sch (KiCad schematic)
At the start: 19 parts, among them U3 LMR33640ADDAR

Commit message: First draft of GSECM schematic
Parts:
- renumbered R3 to R1, R8 to R2, R10 to R3, R11 to R4
Changed lines of the file:
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@@
 		(dnp no)
 		(fields_autoplaced yes)
-		(property "Reference" "R8"
+		(property "Reference" "R2"
 			(at 175.26 104.1399 0)
 			(effects
@@
 			(project "GSECPM"
 				(path "/03409c33-60c4-4fcd-8521-73191969e03b/5aa66df7-1392-47c9-9eac-08ee8ee35544"
-					(reference "R8")
+					(reference "R2")
 					(unit 1)
 				)
@@
 		(on_board yes)
 		(dnp no)
-		(property "Reference" "R10"
+		(property "Reference" "R3"
 			(at 67.056 82.804 0)
 			(effects
@@
 			(project "GSECPM"
 				(path "/03409c33-60c4-4fcd-8521-73191969e03b/5aa66df7-1392-47c9-9eac-08ee8ee35544"
-					(reference "R10")
+					(reference "R3")
 					(unit 1)
 				)
@@
 		(on_board yes)
 		(dnp no)
-		(property "Reference" "R11"
+		(property "Reference" "R4"
 			(at 66.802 71.374 0)
 			(effects
@@
 			(project "GSECPM"
 				(path "/03409c33-60c4-4fcd-8521-73191969e03b/5aa66df7-1392-47c9-9eac-08ee8ee35544"
-					(reference "R11")
+					(reference "R4")
 					(unit 1)
 				)
@@
 		(on_board yes)
 		(dnp no)
-		(property "Reference" "R3"
+		(property "Reference" "R1"
 			(at 166.116 85.344 0)
 			(effects
@@
 			(project "GSECPM"
 				(path "/03409c33-60c4-4fcd-8521-73191969e03b/5aa66df7-1392-47c9-9eac-08ee8ee35544"
-					(reference "R3")
-					(unit 1)
-				)
+					(reference "R1")
+					(unit 1)
+				)
