File: hardware/GSECPM/GSECPM.kicad_sch (KiCad schematic)
At the start: 4 parts, among them J3 PJ-102B

Commit message: First draft of GSECM schematic
Parts:
- removed A1, A2: RaspberryPi_Pico, Module:RaspberryPi_Pico_Common_Unspecified, symbol MCU_Module:RaspberryPi_Pico
- removed C1: 10uF, symbol Device:C
- removed J3: PJ-102B, PJ-102B:CUI_PJ-102B, symbol 12v_barrel_jack:PJ-102B
- added C29, C30, C38: 0.1uF, symbol Device:C
- added J14: Radio Module Connector, Connector_PinHeader_2.54mm:PinHeader_1x04_P2.54mm_Vertical, symbol Connector_Generic:Conn_01x04
- added P2: USB_C_ACT, symbol Connector:USB_C_Plug_USB2.0
- added P3: USB_C_DAQ, symbol Connector:USB_C_Plug_USB2.0
- added R29, R32: 1M, symbol Device:R
- added R30, R31: 5.1k, symbol Device:R
- added R39, R40: 10k, symbol Device:R
- added SW1, SW2, SW3, SW4: SW_Push, symbol Switch:SW_Push
- added U2, U4: STM32F042K6T6, LQFP-32, symbol STM32F042K6T6:STM32F042K6T6
Connections:
- net +5V: now also J14.1 (Pin_1), P2.A4 (VBUS), P2.A9 (VBUS), P2.B4 (VBUS), P2.B9 (VBUS), P3.A4 (VBUS), P3.A9 (VBUS), P3.B4 (VBUS), P3.B9 (VBUS)
- net GND: now also C29.2, C30.2, C38.2, J14.4 (Pin_4), R29.2, R30.2, R31.2, R32.2, R39.2, R40.2, SW2.2, SW3.2, U2.16 (VSS), U2.32 (VSS), U4.16 (VSS), U4.32 (VSS)
- new net: R39.1, SW1.1, U2.31 (PB8-BOOT0)
- new net: P3.A7 (D-), U4.21 (PA11)
- new net: P3.A6 (D+), U4.22 (PA12)
- new net: R40.1, SW4.1, U4.31 (PB8-BOOT0)
- new net: SW3.1, U4.4 (NRST)
- new net: C29.1, P2.A1 (GND), P2.A12 (GND), P2.B1 (GND), P2.B12 (GND), P2.S1 (SHIELD), R29.1
- new net: C30.1, P3.A1 (GND), P3.A12 (GND), P3.B1 (GND), P3.B12 (GND), P3.S1 (SHIELD), R32.1
- new net: P3.A5 (CC), R31.1
- new net: P2.A5 (CC), R30.1
- new net: P2.A6 (D+), U2.22 (PA12)
- new net: P2.A7 (D-), U2.21 (PA11)
- new net: SW2.1, U2.4 (NRST)
- new net +3.3V: C38.1, SW1.2, SW4.2, U2.1 (VDD), U2.17 (VDDIO2), U2.5 (VDDA), U4.1 (VDD), U4.5 (VDDA)
- new net GPIO2 (Radio_UART_TX): J14.2 (Pin_2)
- new net GPIO3 (Radio_UART_RX): J14.3 (Pin_3)
- new net Inputs_DAQ/ADC_CS: U2.6 (PA0)
- new net Inputs_DAQ/SPI_CLK: U2.7 (PA1)
- new net Inputs_DAQ/SPI_MISO: U2.8 (PA2)
- new net Inputs_DAQ/SPI_MOSI: U2.9 (PA3)
- new net Inputs_DAQ/TC1_CS: U2.10 (PA4)
- new net Inputs_DAQ/TC2_CS: U2.11 (PA5)
- new net Inputs_DAQ/TC3_CS: U2.12 (PA6)
- new net MISO(ACT): U4.10 (PA4)
- new net MISO(DAQ): U2.26 (PB3)
- new net MOSI(ACT): U4.9 (PA3)
- new net MOSI(DAQ): U2.27 (PB4)
- new net Outputs_ACT/PB0(Nitrous_Cooling): U4.14 (PB0)
- new net Outputs_ACT/PB1(Internal_Cooling): U4.15 (PB1)
- new net Outputs_ACT/PB3(QD_E-Match): U4.26 (PB3)
- new net Outputs_ACT/PB4(Ignition_E-Match): U4.27 (PB4)
- new net Outputs_ACT/PB5(Fill_Servo1): U4.28 (PB5)
- new net Outputs_ACT/PB6(Fill_Servo2): U4.29 (PB6)
- new net Outputs_ACT/PB7(Purge_Servo): U4.30 (PB7)
- new net PA0(ServoPWR_Switch): U4.6 (PA0)
- new net SCLK(ACT): U4.8 (PA2)
- new net SCLK(DAQ): U2.15 (PB1)
- new net SCSN(ACT): U4.7 (PA1)
- new net SCSN(DAQ): U2.14 (PB0)
- no-connect marks 6 -> 3
Other:
- sheet Ethernet renamed Ethernet_ACT
- removed sheet BuckConverter
- added sheet Ethernet_DAQ (ethernet_daq.kicad_sch)
- added sheet Inputs_DAQ (inputs_daq.kicad_sch)
- added sheet Outputs_ACT (outputs_act.kicad_sch)
- added sheet Power (Power.kicad_sch)
- sheet Ethernet_ACT: file ethernet.kicad_sch -> ethernet_act.kicad_sch
- sheet Ethernet_ACT ports: added MISO(ACT), MOSI(ACT), SCLK(ACT), SCSN(ACT); removed none
- note added: "Radio Module Connection"
