File: hardware/GSECPM/ethernet.kicad_sch (KiCad schematic)
At the start: 6 parts, among them J1 ARJM11D7-114-AB-EW2, J2 ARJM11D7-114-AB-EW2, U1 W5500, U2 W5500, Y1 ASV-25.000MHZ-EJ-T, Y2 ASV-25.000MHZ-EJ-T

Commit message: First draft of GSECM schematic
Parts:
- removed J2: ARJM11D7-114-AB-EW2, CONN_ARJM11D7-114-AB-EW2_ABR, symbol rj45-conn:ARJM11D7-114-AB-EW2
- removed U2: W5500, 48LQFP_W5500_WIZ, symbol W5500:W5500
- removed Y1, Y2: ASV-25.000MHZ-EJ-T, ASV25000MHZEJT, symbol ASV Clock:ASV-25.000MHZ-EJ-T
- added D1, D2: LED, symbol Device:LED
- added R5, R6: 120, symbol Device:R
Connections:
- net +3.3V: now reaches U1.11 (AVDD)
- net +3.3V: now also U1.15 (AVDD), U1.17 (AVDD), U1.21 (AVDD), U1.36 (INTN), U1.37 (RSTN), U1.4 (AVDD), U1.8 (AVDD), R5.1, R6.1
- net GND: now reaches U1.14 (AGND)
- net GND: now also U1.16 (AGND), U1.19 (AGND), U1.29 (GND), U1.3 (AGND), U1.38 (RSVD), U1.39 (RSVD), U1.40 (RSVD), U1.41 (RSVD), U1.42 (RSVD), U1.48 (AGND), U1.9 (AGND)
- net at U1.25 (LINKLED): now also D1.1 (K)
- net at U1.27 (ACTLED): now also D2.1 (K)
- net SCSN(ACT): now reaches U1.32 (SCSN)
- net SCLK(ACT): now reaches U1.33 (SCLK)
- net MISO(ACT): now reaches U1.34 (MISO)
- net MOSI(ACT): now reaches U1.35 (MOSI)
- net PMODE2(ACT): now reaches U1.43 (PMODE2)
- net PMODE1(ACT): now reaches U1.44 (PMODE1)
- net PMODE0(ACT): now reaches U1.45 (PMODE0)
- new net: D2.2 (A), R5.2
- new net: D1.2 (A), R6.2
- no-connect marks 0 -> 2
Other:
- moved on the sheet: J1, U1
